File: PDU_Adapter.kicad_pcb (KiCad board)
At the start: 2 copper layers, 170.2 x 231.1 mm, 6 parts

Commit message: VER1.0: расставил контакторы
Parts:
- added J1: Main_Contactor_Coil, Molex_My:Mini-Fit_01x02_Vertical, F.Cu at (402.7, 315.8)
- added J10: Shunt_2_FeedBack, Molex_My:Mini-Fit_01x02_Vertical, F.Cu at (442.7, 553.7)
- added J11: Conn_01x02, Connector:Banana_Jack_1Pin, F.Cu at (285.1, 311.1)
- added J11: Conn_01x02, Connector:Banana_Jack_1Pin, F.Cu at (589.9, 518.8)
- added J11: Conn_01x02, Connector:Banana_Jack_1Pin, F.Cu at (589.9, 363.2)
- added J2: Precharge_1_Coil, Molex_My:Mini-Fit_01x02_Vertical, F.Cu at (442.0, 315.8)
- added J3: Shunt_1_Coil, Molex_My:Mini-Fit_01x02_Vertical, F.Cu at (442.0, 390.1)
- added J4: Precharge_2_Coil, Molex_My:Mini-Fit_01x02_Vertical, F.Cu at (442.0, 464.4)
- added J5: Sunt_2_Coil, Molex_My:Mini-Fit_01x02_Vertical, F.Cu at (442.7, 538.7)
- added J6: Main_Contactor_FeedBack, Molex_My:Mini-Fit_01x02_Vertical, F.Cu at (402.7, 330.8)
- added J7: Precharge_1_FeedBack, Molex_My:Mini-Fit_01x02_Vertical, F.Cu at (442.0, 330.8)
- added J8: Shunt_1_FeedBack, Molex_My:Mini-Fit_01x02_Vertical, F.Cu at (442.0, 405.1)
- added J9: Precharge_2_FeedBack, Molex_My:Mini-Fit_01x02_Vertical, F.Cu at (442.0, 479.4)
- added R1: R, Resistor_THT:R_Axial_Power_L60.0mm_W14.0mm_P66.04mm, F.Cu at (573.4, 241.3)
- added R10: R, Resistor_THT:R_Axial_Power_L60.0mm_W14.0mm_P66.04mm, B.Cu at (573.4, 264.8)
- added R11: R, Resistor_THT:R_Axial_Power_L60.0mm_W14.0mm_P66.04mm, B.Cu at (573.4, 280.0)
- added R12: R, Resistor_THT:R_Axial_Power_L60.0mm_W14.0mm_P66.04mm, B.Cu at (573.4, 295.3)
- added R13: R, Resistor_THT:R_Axial_Power_L60.0mm_W14.0mm_P66.04mm, B.Cu at (573.4, 310.5)
- added R14: R, Resistor_THT:R_Axial_Power_L60.0mm_W14.0mm_P66.04mm, B.Cu at (573.4, 325.8)
- added R15: R, Resistor_THT:R_Axial_Power_L60.0mm_W14.0mm_P66.04mm, B.Cu at (573.4, 341.0)
- added R16: R, Resistor_THT:R_Axial_Power_L60.0mm_W14.0mm_P66.04mm, F.Cu at (507.4, 394.3)
- added R17: R, Resistor_THT:R_Axial_Power_L60.0mm_W14.0mm_P66.04mm, F.Cu at (507.4, 409.6)
- added R18: R, Resistor_THT:R_Axial_Power_L60.0mm_W14.0mm_P66.04mm, F.Cu at (507.4, 424.8)
- added R19: R, Resistor_THT:R_Axial_Power_L60.0mm_W14.0mm_P66.04mm, F.Cu at (507.4, 440.1)
- added R2: R, Resistor_THT:R_Axial_Power_L60.0mm_W14.0mm_P66.04mm, F.Cu at (573.4, 256.5)
- added R20: R, Resistor_THT:R_Axial_Power_L60.0mm_W14.0mm_P66.04mm, F.Cu at (507.4, 455.3)
- added R21: R, Resistor_THT:R_Axial_Power_L60.0mm_W14.0mm_P66.04mm, F.Cu at (507.4, 470.5)
- added R22: R, Resistor_THT:R_Axial_Power_L60.0mm_W14.0mm_P66.04mm, F.Cu at (507.4, 485.8)
- added R23: R, Resistor_THT:R_Axial_Power_L60.0mm_W14.0mm_P66.04mm, B.Cu at (507.4, 387.4)
- added R24: R, Resistor_THT:R_Axial_Power_L60.0mm_W14.0mm_P66.04mm, B.Cu at (507.4, 402.6)
- added R25: R, Resistor_THT:R_Axial_Power_L60.0mm_W14.0mm_P66.04mm, B.Cu at (507.4, 417.8)
- added R26: R, Resistor_THT:R_Axial_Power_L60.0mm_W14.0mm_P66.04mm, B.Cu at (507.4, 433.1)
- added R27: R, Resistor_THT:R_Axial_Power_L60.0mm_W14.0mm_P66.04mm, B.Cu at (507.4, 448.3)
- added R28: R, Resistor_THT:R_Axial_Power_L60.0mm_W14.0mm_P66.04mm, B.Cu at (507.4, 463.6)
- added R29: R, Resistor_THT:R_Axial_Power_L60.0mm_W14.0mm_P66.04mm, B.Cu at (507.4, 478.8)
- added R3: R, Resistor_THT:R_Axial_Power_L60.0mm_W14.0mm_P66.04mm, F.Cu at (573.4, 271.8)
- added R30: R, Resistor_THT:R_Axial_Power_L60.0mm_W14.0mm_P66.04mm, B.Cu at (507.4, 494.0)
- added R4: R, Resistor_THT:R_Axial_Power_L60.0mm_W14.0mm_P66.04mm, F.Cu at (507.4, 287.0)
- added R5: R, Resistor_THT:R_Axial_Power_L60.0mm_W14.0mm_P66.04mm, F.Cu at (573.4, 302.3)
- added R6: R, Resistor_THT:R_Axial_Power_L60.0mm_W14.0mm_P66.04mm, F.Cu at (573.4, 317.5)
- added R7: R, Resistor_THT:R_Axial_Power_L60.0mm_W14.0mm_P66.04mm, F.Cu at (573.4, 332.7)
- added R8: R, Resistor_THT:R_Axial_Power_L60.0mm_W14.0mm_P66.04mm, B.Cu at (573.4, 234.3)
- added R9: R, Resistor_THT:R_Axial_Power_L60.0mm_W14.0mm_P66.04mm, B.Cu at (573.4, 249.6)
- D3: value EV200 -> ~; footprint Contactor:EV200 -> Sensor_My:YMC15S-500A; moved to B.Cu
- D6: value ~ -> EV200; footprint Sensor_My:YMC15S-500A -> Contactor:EV200
- moved D3 287.4 mm to (332.1, 290.8)
- moved D2 171.1 mm to (473.7, 290.8)
- moved D4 163.6 mm to (473.7, 365.1), turned to 0 degrees
- moved D1 160.7 mm to (384.3, 290.8)
- moved D6 145.4 mm to (474.3, 513.7), turned to 0 degrees
- moved D5 58.8 mm to (473.7, 439.4)
Connections:
- D1 pad A2: unconnected-(D1-PadA2) -> Net-(D1-PadA2)
- D2 pad A1: unconnected-(D2-PadA1) -> Net-(D1-PadA2)
- D2 pad A2: unconnected-(D2-PadA2) -> Net-(D2-PadA2)
- D4 pad A1: unconnected-(D4-PadA1) -> Net-(D1-PadA2)
- D4 pad A2: unconnected-(D4-PadA2) -> VDC+_Invertor
- D5 pad A1: unconnected-(D5-PadA1) -> Net-(D1-PadA2)
- D5 pad A2: unconnected-(D5-PadA2) -> Net-(D5-PadA2)
Routing:
- net Net-(D1-PadA2): track 0.00 -> 305.8 mm
Other:
- board size 170.2 x 231.1 mm -> 266.1 x 339.1 mm
