File: PDU_Adapter.kicad_sch (KiCad schematic)
At the start: 7 parts

Commit message: VER1.0: расставил контакторы
Parts:
- added J1: Main_Contactor_Coil, Molex_My:Mini-Fit_01x02_Vertical, symbol Connector_Generic:Conn_01x02
- added J10: Shunt_2_FeedBack, Molex_My:Mini-Fit_01x02_Vertical, symbol Connector_Generic:Conn_01x02
- added J11: Conn_01x02, Connector:Banana_Jack_1Pin, symbol Connector_Generic:Conn_01x02
- added J2: Precharge_1_Coil, Molex_My:Mini-Fit_01x02_Vertical, symbol Connector_Generic:Conn_01x02
- added J3: Shunt_1_Coil, Molex_My:Mini-Fit_01x02_Vertical, symbol Connector_Generic:Conn_01x02
- added J4: Precharge_2_Coil, Molex_My:Mini-Fit_01x02_Vertical, symbol Connector_Generic:Conn_01x02
- added J5: Sunt_2_Coil, Molex_My:Mini-Fit_01x02_Vertical, symbol Connector_Generic:Conn_01x02
- added J6: Main_Contactor_FeedBack, Molex_My:Mini-Fit_01x02_Vertical, symbol Connector_Generic:Conn_01x02
- added J7: Precharge_1_FeedBack, Molex_My:Mini-Fit_01x02_Vertical, symbol Connector_Generic:Conn_01x02
- added J8: Shunt_1_FeedBack, Molex_My:Mini-Fit_01x02_Vertical, symbol Connector_Generic:Conn_01x02
- added J9: Precharge_2_FeedBack, Molex_My:Mini-Fit_01x02_Vertical, symbol Connector_Generic:Conn_01x02
- added R1, R10, R12, R13, R14, R15, R16, R17, R18, R19, R2, R20, R21, R22, R23, R24, R25, R26, R27, R28, R29, R3, R30, R4, R5, R6, R7, R8, R9: R, Resistor_THT:R_Axial_Power_L60.0mm_W14.0mm_P66.04mm, symbol Device:R
- R11: renamed from R1; footprint (none) -> Resistor_THT:R_Axial_Power_L60.0mm_W14.0mm_P66.04mm
- renumbered D6 to D3, D3 to D4, D4 to D5, D5 to D6
Connections:
- net at D1.A2: now also D2.A1, D4.A1, D5.A1, D6.A1
- net at D1.A3: now also J6.2 (Pin_2)
- net at D1.A4: now also J6.1 (Pin_1)
- net at D1.C1: now also J1.1 (Pin_1)
- net at D1.C2: now also J1.2 (Pin_2)
- net VDC+_Invertor: now reaches D4.A2
- net VDC+_Invertor: now also R11.2, R1.2, R10.2, R12.2, R13.2, R14.2, R15.2, R2.2, R3.2, R4.2, R5.2, R6.2, R7.2, R8.2, R9.2
- net at D4.A3: now also J8.2 (Pin_2)
- net at D4.A4: now also J8.1 (Pin_1)
- net at D4.C1: now also J3.1 (Pin_1)
- net at D4.C2: now also J3.2 (Pin_2)
- net at D2.A2: now also R11.1, R1.1, R10.1, R12.1, R13.1, R14.1, R15.1, R2.1, R3.1, R4.1, R5.1, R6.1, R7.1, R8.1, R9.1
- net at D2.A3: now also J7.2 (Pin_2)
- net at D2.A4: now also J7.1 (Pin_1)
- net at D2.C1: now also J2.1 (Pin_1)
- net at D2.C2: now also J2.2 (Pin_2)
- net VDC+_ECG: now reaches D6.A2
- net VDC+_ECG: now also R16.2, R17.2, R18.2, R19.2, R20.2, R21.2, R22.2, R23.2, R24.2, R25.2, R26.2, R27.2, R28.2, R29.2, R30.2
- net at D6.A3: now also J10.2 (Pin_2)
- net at D6.A4: now also J10.1 (Pin_1)
- net at D6.C1: now also J5.1 (Pin_1)
- net at D6.C2: now also J5.2 (Pin_2)
- net at D5.A2: now also R16.1, R17.1, R18.1, R19.1, R20.1, R21.1, R22.1, R23.1, R24.1, R25.1, R26.1, R27.1, R28.1, R29.1, R30.1
- net at D5.A3: now also J9.2 (Pin_2)
- net at D5.A4: now also J9.1 (Pin_1)
- net at D5.C1: now also J4.1 (Pin_1)
- net at D5.C2: now also J4.2 (Pin_2)
Other:
- moved on the sheet: D1, D2, D3, D4, D5, D6, R11
